Commit message: Finally got foxglove working, now visulizes vehicle controls, the lidar points, camera, and plots the steering. Still working on getting the lane path and the 3d model to show up

File: beamng_sim/foxglove_integration/model/bmw_x5/bmw_x5.urdf (robot description, URDF)
Before this commit: robot bmw_x5, 5 links, 5 joints
Links:
- link body: geometry visual mesh filename=file:///c:/Users/user/Documents/github/self-driving-car-sim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
- link front_left_wheel: geometry visual mesh filename=file:///c:/Users/user/Documents/github/self-driving-car-sim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
- link front_right_wheel: geometry visual mesh filename=file:///c:/Users/user/Documents/github/self-driving-car-sim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
- link rear_left_wheel: geometry visual mesh filename=file:///c:/Users/user/Documents/github/self-driving-car-sim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
- link rear_right_wheel: geometry visual mesh filename=file:///c:/Users/user/Documents/github/self-driving-car-sim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
Joints:
- removed joint body_root_joint
- joint front_left_wheel_joint: axis 0 1 0 -> (none); type revolute -> fixed
- joint front_right_wheel_joint: axis 0 1 0 -> (none); type revolute -> fixed
- joint rear_left_wheel_joint: axis 0 1 0 -> (none); type revolute -> fixed
- joint rear_right_wheel_joint: axis 0 1 0 -> (none); type revolute -> fixed
